Commit message: Change model name

File: urdf/thunder_line_follower.urdf (robot description, URDF)
Before this commit: robot modelo_carrinho, 13 links, 12 joints
Links:
- link arduino_link: geometry collision mesh filename=package://thunder_line_follower_pmr3100/meshes/arduino_link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; visual mesh filename=package://thunder_line_follower_pmr3100/meshes/arduino_link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
- link base_link: geometry collision mesh filename=package://thunder_line_follower_pmr3100/meshes/base_link.stl; visual mesh filename=package://thunder_line_follower_pmr3100/meshes/base_link.stl
- link bateria_link: geometry collision mesh filename=package://thunder_line_follower_pmr3100/meshes/bateria_link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; visual mesh filename=package://thunder_line_follower_pmr3100/meshes/bateria_link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
- link line1_link: geometry collision mesh filename=package://thunder_line_follower_pmr3100/meshes/line1_link.s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; visual mesh filename=package://thunder_line_follower_pmr3100/meshes/line1_link.s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
- link line2_link: geometry collision mesh filename=package://thunder_line_follower_pmr3100/meshes/line2_link.s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; visual mesh filename=package://thunder_line_follower_pmr3100/meshes/line2_link.s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
- link line3_link: geometry collision mesh filename=package://thunder_line_follower_pmr3100/meshes/line3_link.s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; visual mesh filename=package://thunder_line_follower_pmr3100/meshes/line3_link.s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
- link line4_link: geometry collision mesh filename=package://thunder_line_follower_pmr3100/meshes/line4_link.s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; visual mesh filename=package://thunder_line_follower_pmr3100/meshes/line4_link.s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
- link line5_link: geometry collision mesh filename=package://thunder_line_follower_pmr3100/meshes/line5_link.s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; visual mesh filename=package://thunder_line_follower_pmr3100/meshes/line5_link.s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
- link motordireito_link: geometry collision mesh filename=package://thunder_line_follower_pmr3100/meshes/motordireito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; visual mesh filename=package://thunder_line_follower_pmr3100/meshes/motordireito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
- link motoresquerdo_link: geometry collision mesh filename=package://thunder_line_follower_pmr3100/meshes/motoresquerd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; visual mesh filename=package://thunder_line_follower_pmr3100/meshes/motoresquerd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
- link rodadireita_link: geometry collision mesh filename=package://thunder_line_follower_pmr3100/meshes/rodadireita_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; visual mesh filename=package://thunder_line_follower_pmr3100/meshes/rodadireita_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
- link rodaesquerda_link: geometry collision mesh filename=package://thunder_line_follower_pmr3100/meshes/rodaesquerda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; visual mesh filename=package://thunder_line_follower_pmr3100/meshes/rodaesquerda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
- link sonar_link: geometry collision mesh filename=package://thunder_line_follower_pmr3100/meshes/sonar_link.s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; visual mesh filename=package://thunder_line_follower_pmr3100/meshes/sonar_link.s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

File: urdf/thunder_line_follower.xacro (robot description, xacro)
@@ -1,14 +1,14 @@
 <?xml version="1.0" encoding="utf-8"?>
-<robot name="modelo_carrinho"
+<robot name="thunder_line_follower_pmr3100"
   xmlns:xacro="http://www.ros.org/wiki/xacro">
  <!-- Global argument used in .gazebo file to set sensor visual properties -->
   <xacro:arg name="debug_sensors" default="false" />
   <!-- Import all Gazebo plugins -->
-  <xacro:include filename="$(find modelo_carrinho)/urdf/modelo_carrinho.gazebo" />
+  <xacro:include filename="$(find thunder_line_follower_pmr3100)/urdf/thunder_line_follower_pmr3100.gazebo" />
   <!-- Code exported from SolidWorks -->
-  <xacro:include filename="$(find modelo_carrinho)/urdf/modelo_carrinho.urdf" />
+  <xacro:include filename="$(find thunder_line_follower_pmr3100)/urdf/thunder_line_follower_pmr3100.urdf" />
   <!-- Definition of motor -->
-  <xacro:include filename="$(find modelo_carrinho)/urdf/motor.xacro"/>
-  <xacro:include filename="$(find modelo_carrinho)/urdf/colors.xacro"/>
+  <xacro:include filename="$(find thunder_line_follower_pmr3100)/urdf/motor.xacro"/>
+  <xacro:include filename="$(find thunder_line_follower_pmr3100)/urdf/colors.xacro"/>
   <xacro:motor joint_name="rodaesquerda" gear_rate="1"/>
   <xacro:motor joint_name="rodadireita" gear_rate="1"/>
